Commit message: camera model added with sensor for realsense

File: robot/xarm_description/urdf/lite6/lite6.gazebo.xacro (robot description, xacro)
@@ -23,4 +23,53 @@
       <selfCollide>true</selfCollide>
     </gazebo>
+    <gazebo reference="${prefix}realsense_camera">
+      <sensor name="realsense_d435" type="rgbd_camera">
+        <pose>0 0 0 0 0 -1.571</pose>
+        <update_rate>60</update_rate>
+        <camera name="camera">
+          <horizontal_fov>1.0472</horizontal_fov>
+          <lens>
+            <intrinsics>
+              <!-- fx = fy = width / ( 2 * tan (hfov / 2 ) ) -->
+              <fx>554.25469</fx>
+              <fy>554.25469</fy>
+              <!-- cx = ( width + 1 ) / 2 -->
+              <cx>320.5</cx>
+              <!-- cy = ( height + 1 ) / 2 -->
+              <cy>240.5</cy>
+              <s>0</s>
+            </intrinsics>
+          </lens>
+          <distortion>
+            <k1>0.0</k1>
+            <k2>0.0</k2>
+            <k3>0.0</k3>
+            <p1>0.0</p1>
+            <p2>0.0</p2>
+            <center>0.5 0.5</center>
+          </distortion>
+          <image>
+            <width>640</width>
+            <height>480</height>
+            <format>R8G8B8</format>
+          </image>
+          <clip>
+            <near>0.01</near>
+            <far>300</far>
+          </clip>
+          <depth_camera>
+            <clip>
+              <near>0.1</near>
+              <far>10</far>
+            </clip>
+          </depth_camera>
+          <noise>
+            <type>gaussian</type>
+            <mean>0</mean>
+            <stddev>0.007</stddev>
+          </noise>
+        </camera>
+      </sensor>
+    </gazebo>
   </xacro:macro>
 </robot>

File: robot/xarm_description/urdf/lite6/lite6.urdf.xacro (robot description, xacro)
@@ -213,4 +213,49 @@
       <child link="${prefix}link_eef" />
     </joint> -->
+    <!-- create link for the camera and connect joint to world frame -->
+    <link name="${prefix}realsense_camera">
+      <inertial>
+        <mass value="0.0615752" />
+        <inertia
+        ixx="9.108e-05"
+        ixy="0"
+        ixz="0"
+        iyy="2.51e-06"
+        iyz="0"
+        izz="8.931e-05" />
+        <origin xyz="0 0 0" rpy="0 0 0" />
+      </inertial>
+      <visual>
+        <origin
+          xyz="0 0 0"
+          rpy="0 0 0" />
+        <geometry>
+          <mesh
+            filename="$(find xarm_description)/meshes/camera/realsense/meshes/realsense.dae" />
+        </geometry>
+        <material
+          name="">
+          <color rgba="0.760 0.564 0.403 1" />
+        </material>
+      </visual>
+      <collision>
+      <origin
+        xyz="0 0 0"
+        rpy="0 0 0" />
+      <geometry>
+        <mesh
+          filename="$(find xarm_description)/meshes/camera/realsense/meshes/realsense.dae" />
+      </geometry>
+      <material
+        name="">
+        <color rgba="0.760 0.564 0.403 1" />
+      </material>
+    </collision>
+    </link>
+    <joint name="camera_world" type="fixed">
+      <origin xyz="0.11 0 1.25" rpy="1.571 0 1.571" />
+      <parent link="world" />
+      <child link="realsense_camera" />
+    </joint>
   </xacro:macro>
 </robot>

Commit message: sensor param & camera joint modified

File: robot/xarm_description/urdf/lite6/lite6.gazebo.xacro (robot description, xacro)
@@ -25,5 +25,5 @@
     <gazebo reference="${prefix}realsense_camera">
       <sensor name="realsense_d435" type="rgbd_camera">
-        <pose>0 0 0 0 0 -1.571</pose>
+        <pose>0 0 0 4.71 4.71 0</pose>
         <update_rate>60</update_rate>
         <camera name="camera">
@@ -32,10 +32,10 @@
             <intrinsics>
               <!-- fx = fy = width / ( 2 * tan (hfov / 2 ) ) -->
-              <fx>554.25469</fx>
-              <fy>554.25469</fy>
+              <fx>931.1829833984375</fx>
+              <fy>931.1829833984375</fy>
               <!-- cx = ( width + 1 ) / 2 -->
-              <cx>320.5</cx>
+              <cx>640</cx>
               <!-- cy = ( height + 1 ) / 2 -->
-              <cy>240.5</cy>
+              <cy>360</cy>
               <s>0</s>
             </intrinsics>
@@ -50,6 +50,6 @@
           </distortion>
           <image>
-            <width>640</width>
-            <height>480</height>
+            <width>1280</width>
+            <height>720</height>
             <format>R8G8B8</format>
           </image>

File: robot/xarm_description/urdf/lite6/lite6.urdf.xacro (robot description, xacro)
@@ -254,5 +254,5 @@
     </link>
     <joint name="camera_world" type="fixed">
-      <origin xyz="0.11 0 1.25" rpy="1.571 0 1.571" />
+      <origin xyz="0.11 0 1.25" rpy="3.14 0 1.57" />
       <parent link="world" />
       <child link="realsense_camera" />
